File: kicad/esp_music_vis/esp_music_vis.kicad_pcb (KiCad board)
At the start: 2 copper layers, 100 x 100 mm, 2 parts, among them U1 ESP32_WROOM_32D_devkit

Commit message: PCB first version
Parts:
- removed PWR1: Conn_01x03_Male, Connector_PinHeader_2.54mm:PinHeader_1x03_P2.54mm_Vertical
- added ?: , , F.Cu at (98.6, 51.9)
- added ?: , , F.Cu at (102.3, 57.0)
- added ?: , , F.Cu at (57.3, 62.0)
- added ?: , , F.Cu at (51.7, 61.1)
- added ?: , , F.Cu at (57.3, 67.0)
- added ?: , , F.Cu at (57.3, 77.0)
- added ?: , , F.Cu at (148.9, 55.2)
- added ?: , , F.Cu at (98.6, 54.9)
- added ?: , , F.Cu at (57.3, 72.0)
- added ?: , , F.Cu at (148.4, 56.2)
- added ?: , , B.Cu at (148.4, 76.2)
- added ?: , , F.Cu at (98.6, 57.0)
- added ?: , , B.Cu at (148.4, 73.7)
- added ?: , , B.Cu at (148.4, 53.8)
- added ?: , , B.Cu at (148.4, 71.1)
- added ?: , , B.Cu at (51.7, 76.2)
- added ?: , , B.Cu at (51.7, 53.7)
- added ?: , , B.Cu at (148.4, 61.1)
- added ?: , , B.Cu at (148.4, 51.2)
- added ?: , , B.Cu at (51.7, 63.7)
- added ?: , , B.Cu at (148.4, 63.6)
- added ?: , , B.Cu at (51.6, 66.2)
- added ?: , , F.Cu at (57.3, 64.5)
- added ?: , , B.Cu at (51.7, 73.7)
- added ?: , , B.Cu at (148.4, 66.2)
- added ?: , , B.Cu at (51.7, 56.2)
- added ?: , , B.Cu at (51.7, 71.2)
- added ?: , , F.Cu at (102.3, 54.9)
- added ?: , , F.Cu at (102.3, 51.9)
- added ?: , , F.Cu at (51.7, 51.1)
- added ?: , , F.Cu at (148.9, 65.1)
- added ?: , , F.Cu at (51.1, 55.0)
- added ?: , , F.Cu at (57.3, 74.5)
- added D1: LED, LED_THT:LED_D5.0mm_Clear, F.Cu at (64.3, 143.6)
- added D2: LED, LED_THT:LED_D5.0mm_Clear, F.Cu at (72.5, 143.6)
- added D3: LED, LED_THT:LED_D5.0mm_Clear, F.Cu at (80.7, 143.6)
- added D4: LED, LED_THT:LED_D5.0mm_Clear, F.Cu at (88.9, 143.6)
- added J1: Conn_01x02_Pin, Connector_AMASS:AMASS_XT30UPB-M_1x02_P5.0mm_Vertical, F.Cu at (144.8, 111.7)
- added J2: Conn_01x03_Pin, Connector_PinHeader_2.54mm:PinHeader_1x03_P2.54mm_Vertical, F.Cu at (54.1, 140.1)
- added J3: Conn_01x03_Pin, Connector_PinHeader_2.54mm:PinHeader_1x03_P2.54mm_Vertical, F.Cu at (59.6, 140.1)
- added J4: Conn_01x03_Pin, Connector_Phoenix_MC_HighVoltage:PhoenixContact_MCV_1,5_3-G-5.08_1x03_P5.08mm_Vertical, F.Cu at (138.2, 95.1)
- added J4: Conn_01x03_Pin, Connector_Phoenix_MC_HighVoltage:PhoenixContact_MCV_1,5_3-G-5.08_1x03_P5.08mm_Vertical, F.Cu at (53.4, 107.4)
- added J4: Conn_01x03_Pin, Connector_Phoenix_MC_HighVoltage:PhoenixContact_MCV_1,5_3-G-5.08_1x03_P5.08mm_Vertical, F.Cu at (61.8, 84.9)
- added R1: R_Photo, OptoDevice:R_LDR_5.0x4.1mm_P3mm_Vertical, F.Cu at (91.9, 117.6)
- added R2: 260, Resistor_THT:R_Axial_DIN0207_L6.3mm_D2.5mm_P10.16mm_Horizontal, F.Cu at (72.8, 136.1)
- added R3: 260, Resistor_THT:R_Axial_DIN0207_L6.3mm_D2.5mm_P10.16mm_Horizontal, F.Cu at (76.8, 136.1)
- added R4: 260, Resistor_THT:R_Axial_DIN0207_L6.3mm_D2.5mm_P10.16mm_Horizontal, F.Cu at (80.8, 136.1)
- added R5: 260, Resistor_THT:R_Axial_DIN0207_L6.3mm_D2.5mm_P10.16mm_Horizontal, F.Cu at (84.9, 136.1)
- added R6: 10k, Resistor_THT:R_Axial_DIN0207_L6.3mm_D2.5mm_P10.16mm_Horizontal, F.Cu at (88.8, 136.1)
- added R7: 10k, Resistor_THT:R_Axial_DIN0207_L6.3mm_D2.5mm_P10.16mm_Horizontal, F.Cu at (59.2, 124.6)
- added R8: 5.1k, Resistor_THT:R_Axial_DIN0207_L6.3mm_D2.5mm_P10.16mm_Horizontal, F.Cu at (54.2, 134.9)
- added REF**: PAD_11x2, Library:PAD_11x2, F.Cu at (124.4, 149.1)
- added REF**: PAD_11x2, Library:PAD_11x2, F.Cu at (51.8, 65.0)
- added REF**: PAD_2X3, Library:PAD_2X3, F.Cu at (129.1, 90.1)
- added REF** (x3): PAD_2X3, Library:PAD_2X3, F.Cu at (72.3, 90.1)
- added REF**: PAD_11x2, Library:PAD_11x2, F.Cu at (140.7, 149.1)
- added REF** (x3): PAD_2X3, Library:PAD_2X3, F.Cu at (127.7, 90.1)
- added REF** (x3): PAD_2X3, Library:PAD_2X3, F.Cu at (100.0, 90.1)
- added REF**: PAD_11x2, Library:PAD_11x2, F.Cu at (149.7, 75.1)
- added REF**: PAD_2X3, Library:PAD_2X3, F.Cu at (101.5, 90.1)
- added REF**: PAD_11x2, Library:PAD_11x2, F.Cu at (51.9, 75.0)
- added REF**: PAD_11x2, Library:PAD_11x2, F.Cu at (126.7, 93.0)
- added REF**: PAD_2X3, Library:PAD_2X3, B.Cu at (151.4, 74.9)
- added REF**: PAD_2X3, Library:PAD_2X3, B.Cu at (151.4, 55.0)
- added REF**: PAD_2X3, Library:PAD_2X3, B.Cu at (54.6, 65.0)
- added REF**: PAD_2X3, Library:PAD_2X3, B.Cu at (151.4, 64.9)
- added REF**: PAD_2X3, Library:PAD_2X3, B.Cu at (54.7, 75.0)
- added REF**: PAD_2X3, Library:PAD_2X3, B.Cu at (54.7, 55.0)
- added REF**: PAD_11x2, Library:PAD_11x2, F.Cu at (108.1, 149.1)
- added REF**: PAD_11x2, Library:PAD_11x2, F.Cu at (99.1, 93.0)
- added REF**: PAD_2X3, Library:PAD_2X3, F.Cu at (73.7, 90.1)
- added REF**: PAD_11x2, Library:PAD_11x2, F.Cu at (71.3, 93.0)
- moved U1 2.93 mm to (142.1, 129.7)
Connections:
- U1 pad 10: unconnected-(U1-Pad10) -> TOUCH_3
- U1 pad 11: unconnected-(U1-Pad11) -> MOTION
- U1 pad 12: unconnected-(U1-Pad12) -> L_SENSOR
- U1 pad 14: unconnected-(U1-Pad14) -> GND
- U1 pad 15: unconnected-(U1-Pad15) -> +5V
- U1 pad 20: unconnected-(U1-Pad20) -> LED1
- U1 pad 21: unconnected-(U1-Pad21) -> LED2
- U1 pad 22: unconnected-(U1-Pad22) -> LED3
- U1 pad 23: unconnected-(U1-Pad23) -> LED4
- U1 pad 26: unconnected-(U1-Pad26) -> LED_DOUT
- U1 pad 29: (no net) -> GND
- U1 pad 30: (no net) -> +3.3V
- U1 pad 6: unconnected-(U1-Pad6) -> TOUCH_1
- U1 pad 7: unconnected-(U1-Pad7) -> TOUCH_2
Routing:
- net +5V: track 0.00 -> 575.5 mm, vias 0 -> 7
- net GND: track 0.00 -> 471.0 mm, vias 0 -> 7
- net DOUT_2: track 0.00 -> 194.0 mm
- net LED_DOUT: track 0.00 -> 133.5 mm, vias 0 -> 1
- net +3.3V: track 0.00 -> 109.2 mm, vias 0 -> 1
- net MOTION: track 0.00 -> 99.4 mm, vias 0 -> 1
- net L_SENSOR: track 0.00 -> 66.9 mm
- net LED1: track 0.00 -> 61.7 mm
- net LED2: track 0.00 -> 56.9 mm
- net LED3: track 0.00 -> 50.9 mm
- net DOUT1: track 0.00 -> 49.5 mm
- net DIN_4: track 0.00 -> 48.6 mm, vias 0 -> 1
- net DIN_3: track 0.00 -> 47.9 mm, vias 0 -> 1
- net LED4: track 0.00 -> 43.9 mm
- net TOUCH_3: track 0.00 -> 42.9 mm, vias 0 -> 2
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- added copper zone on B.Cu, net +5V
- added copper zone on B.Cu, net GND
- added copper zone on F.Cu, net GND
Other:
- outline, holes or cut-outs redrawn
- board text added: "LDR"
- board text added: "Pawel Wawrow Dawid Godula"
- board text added: "REF**"
- board text added: "T1"
- board text added: "T2"
- board text added: "T3"

Commit message: working-good music visualization, changing settings of vis to be added
Other:
- outline, holes or cut-outs redrawn
Changed lines of the file:
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@@
 		)
 		(property "Value" "LED"
-			(at 1.27 3.96 360)
+			(at 1.27 3.96 0)
 			(layer "F.Fab")
 			(effects
@@
 		)
 		(property "Footprint" "LED_THT:LED_D5.0mm_Clear"
-			(at 0 0 360)
+			(at 0 0 0)
 			(layer "F.Fab")
 			(hide yes)
@@
 		)
 		(property "Datasheet" ""
-			(at 0 0 360)
+			(at 0 0 0)
 			(layer "F.Fab")
 			(hide yes)
@@
 		)
 		(property "Description" ""
-			(at 0 0 360)
+			(at 0 0 0)
 			(layer "F.Fab")
 			(hide yes)
@@
 		)
 		(fp_text user "${REFERENCE}"
-			(at 1.27 0 360)
+			(at 1.27 0 0)
 			(layer "F.Fab")
 			(effects
@@
 		)
 		(property "Value" "LED"
-			(at 1.27 3.96 360)
+			(at 1.27 3.96 0)
 			(layer "F.Fab")
 			(effects
@@
 		)
 		(property "Footprint" "LED_THT:LED_D5.0mm_Clear"
-			(at 0 0 360)
+			(at 0 0 0)
 			(layer "F.Fab")
 			(hide yes)
@@
 		)
 		(property "Datasheet" ""
-			(at 0 0 360)
+			(at 0 0 0)
 			(layer "F.Fab")
 			(hide yes)
@@
 		)
 		(property "Description" ""
-			(at 0 0 360)
+			(at 0 0 0)
 			(layer "F.Fab")
 			(hide yes)
@@
 		)
 		(fp_text user "${REFERENCE}"
-			(at 1.27 0 360)
+			(at 1.27 0 0)
 			(layer "F.Fab")
 			(effects
@@
 		(tags "Resistor LDR5x4.1mm")
 		(property "Reference" "R1"
-			(at 1.5 -2.9 360)
+			(at 1.5 -2.9 0)
 			(layer "F.SilkS")
 			(effects
@@
 		)
 		(property "Value" "R_Photo"
-			(at 1.3 3 360)
+			(at 1.3 3 0)
 			(layer "F.Fab")
 			(effects
@@
 		)
 		(property "Footprint" "OptoDevice:R_LDR_5.0x4.1mm_P3mm_Vertical"
-			(at 0 0 360)
+			(at 0 0 0)
 			(layer "F.Fab")
 			(hide yes)
@@
 		)
 		(property "Datasheet" ""
-			(at 0 0 360)
+			(at 0 0 0)
 			(layer "F.Fab")
 			(hide yes)
@@
 		)
 		(property "Description" ""
-			(at 0 0 360)
+			(at 0 0 0)
 			(layer "F.Fab")
 			(hide yes)
@@
 		)
 		(fp_text user "${REFERENCE}"
-			(at 1.5 -2.9 360)
+			(at 1.5 -2.9 0)
 			(layer "F.Fab")
 			(effects
@@
 		)
 		(property "Value" "LED"
-			(at 1.27 3.96 360)
+			(at 1.27 3.96 0)
 			(layer "F.Fab")
 			(effects
@@
 		)
 		(property "Footprint" "LED_THT:LED_D5.0mm_Clear"
-			(at 0 0 360)
+			(at 0 0 0)
 			(layer "F.Fab")
 			(hide yes)
@@
 		)
 		(property "Datasheet" ""
-			(at 0 0 360)
+			(at 0 0 0)
 			(layer "F.Fab")
 			(hide yes)
@@
 		)
 		(property "Description" ""
-			(at 0 0 360)
+			(at 0 0 0)
 			(layer "F.Fab")
 			(hide yes)
@@
 		)
 		(fp_text user "${REFERENCE}"
-			(at 1.27 0 360)
+			(at 1.27 0 0)
 			(layer "F.Fab")
 			(effects
@@
 		)
 		(property "Value" "LED"
-			(at 1.27 3.96 360)
+			(at 1.27 3.96 0)
 			(layer "F.Fab")
 			(effects
@@
 		)
 		(property "Footprint" "LED_THT:LED_D5.0mm_Clear"
-			(at 0 0 360)
+			(at 0 0 0)
 			(layer "F.Fab")
 			(hide yes)
@@
 		)
 		(property "Datasheet" ""
-			(at 0 0 360)
+			(at 0 0 0)
 			(layer "F.Fab")
 			(hide yes)
@@
 		)
 		(property "Description" ""
-			(at 0 0 360)
+			(at 0 0 0)
 			(layer "F.Fab")
 			(hide yes)
@@
 		)
 		(fp_text user "${REFERENCE}"
-			(at 1.27 0 360)
+			(at 1.27 0 0)
 			(layer "F.Fab")
 			(effects
@@
 		(layer "F.SilkS")
 	)
+	(gr_rect
+		(start 66.8 88.9625)
+		(end 77.8 90.9625)
+		(stroke
+			(width 0.1)
+			(type default)
+		)
+		(fill none)
+		(layer "F.SilkS")
+	)
 	(gr_line
 		(start 81.7 95.9)
@@
 		(layer "F.SilkS")
 	)
+	(gr_rect
+		(start 122.15 88.9625)
+		(end 133.15 90.9625)
+		(stroke
+			(width 0.1)
+			(type default)
+		)
+		(fill none)
+		(layer "F.SilkS")
+	)
 	(gr_line
 		(start 66.75 100)
@@
 		(layer "F.SilkS")
 	)
+	(gr_rect
+		(start 94.55 88.9625)
+		(end 105.55 90.9625)
+		(stroke
+			(width 0.1)
+			(type default)
+		)
+		(fill none)
+		(layer "F.SilkS")
+	)
 	(gr_line
 		(start 150 100)
@@
 	)
 	(gr_circle
+		(center 72.210051 90)
+		(end 72.910051 90.7)
+		(stroke
+			(width 0.1)
+			(type default)
+		)
+		(fill none)
+		(layer "Edge.Cuts")
+	)
+	(gr_circle
 		(center 80.7 116.8)
 		(end 82.4 116.8)
@@
 		(layer "Edge.Cuts")
 	)
-	(gr_line
-		(start 150 70)
-		(end 50 70)
+	(gr_circle
+		(center 76.810051 89.9625)
+		(end 77.510051 90.6625)
 		(stroke
 			(width 0.1)
 			(type default)
 		)
+		(fill none)
 		(layer "Edge.Cuts")
 	)
-	(gr_rect
-		(start 66.8 88.9625)
-		(end 77.8 90.9625)
+	(gr_circle
+		(center 132.160051 89.9625)
+		(end 132.860051 90.6625)
+		(stroke
+			(width 0.1)
+			(type default)
+		)
+		(fill none)
+		(layer "Edge.Cuts")
+	)
+	(gr_circle
+		(center 100.010051 90)
+		(end 100.710051 90.7)
 		(stroke
 			(width 0.1)
@@
 		(layer "Edge.Cuts")
 	)
-	(gr_rect
-		(start 122.15 88.9625)
-		(end 133.15 90.9625)
+	(gr_circle
+		(center 127.768435 89.994316)
+		(end 128.468435 90.694316)
 		(stroke
 			(width 0.1)
@@
 		(layer "Edge.Cuts")
 	)
-	(gr_line
-		(start 150 80)
-		(end 50 80)
+	(gr_circle
+		(center 95.610051 90)
+		(end 96.310051 90.7)
 		(stroke
 			(width 0.1)
 			(type default)
 		)
+		(fill none)
 		(layer "Edge.Cuts")
 	)
-	(gr_line
-		(start 150 100)
-		(end 50 100)
+	(gr_circle
+		(center 123.2 89.989949)
+		(end 123.9 90.689949)
 		(stroke
 			(width 0.1)
 			(type default)
 		)
+		(fill none)
 		(layer "Edge.Cuts")
 	)
@@
 		(layer "Edge.Cuts")
 	)
-	(gr_line
-		(start 150 60)
-		(end 50 60)
+	(gr_circle
+		(center 104.560051 89.9625)
+		(end 105.260051 90.6625)
 		(stroke
 			(width 0.1)
 			(type default)
 		)
+		(fill none)
 		(layer "Edge.Cuts")
 	)
 	(gr_circle
-		(center 144.2 90)
-		(end 145.9 90)
+		(center 67.810051 90)
+		(end 68.510051 90.7)
 		(stroke
 			(width 0.1)
@@
 		(layer "Edge.Cuts")
 	)
-	(gr_rect
-		(start 94.55 88.9625)
-		(end 105.55 90.9625)
+	(gr_circle
+		(center 144.2 90)
+		(end 145.9 90)
 		(stroke
 			(width 0.1)
