File: kicad/esp_music_vis/esp_music_vis.kicad_sch (KiCad schematic)
At the start: 2 parts

Commit message: PCB first version
Parts:
- removed PWR: Conn_01x03_Male, Connector_PinHeader_2.54mm:PinHeader_1x03_P2.54mm_Vertical, symbol Connector:Conn_01x03_Male
- added D1, D2, D3, D4: LED, LED_THT:LED_D5.0mm_Clear, symbol Device:LED
- added J1: Conn_01x02_Pin, Connector_AMASS:AMASS_XT30UPB-M_1x02_P5.0mm_Vertical, symbol Connector:Conn_01x02_Pin
- added J2, J3: Conn_01x03_Pin, Connector_PinHeader_2.54mm:PinHeader_1x03_P2.54mm_Vertical, symbol Connector:Conn_01x03_Pin
- added J4: Conn_01x03_Pin, Connector_Phoenix_MC_HighVoltage:PhoenixContact_MCV_1,5_3-G-5.08_1x03_P5.08mm_Vertical, symbol Connector:Conn_01x03_Pin
- added R1: R_Photo, OptoDevice:R_LDR_5.0x4.1mm_P3mm_Vertical, symbol Device:R_Photo
- added R2, R3, R4, R5: 260, Resistor_THT:R_Axial_DIN0207_L6.3mm_D2.5mm_P10.16mm_Horizontal, symbol Device:R
- added R6, R7: 10k, Resistor_THT:R_Axial_DIN0207_L6.3mm_D2.5mm_P10.16mm_Horizontal, symbol Device:R
- added R8: 5.1k, Resistor_THT:R_Axial_DIN0207_L6.3mm_D2.5mm_P10.16mm_Horizontal, symbol Device:R
- gave numbers to parts that had none: 1
Connections:
- net TOUCH_3: now reaches U1.10 (D27)
- net MOTION: now reaches U1.11 (D14)
- net MOTION: now also J2.2 (Pin_2), R7.2, R8.1
- net L_SENSOR: now reaches U1.12 (D12)
- net L_SENSOR: now also R1.2, R6.1
- net GND: now reaches U1.14 (GND)
- net GND: now also U1.29 (GND), J1.1 (Pin_1), J2.3 (Pin_3), J3.3 (Pin_3), J4.1 (Pin_1), R2.2, R3.2, R4.2, R5.2, R6.2, R7.1
- net +5V: now reaches U1.15 (VIN)
- net +5V: now also J1.2 (Pin_2), J3.1 (Pin_1), J4.3 (Pin_3)
- net LED1: now reaches U1.20 (D21)
- net LED1: now also D1.2 (A)
- net LED2: now reaches U1.21 (D19)
- net LED2: now also D2.2 (A)
- net LED3: now reaches U1.22 (D18)
- net LED3: now also D3.2 (A)
- net LED4: now reaches U1.23 (D5)
- net LED4: now also D4.2 (A)
- net LED_DOUT: now reaches U1.26 (D4)
- net LED_DOUT: now also J4.2 (Pin_2)
- net TOUCH_1: now reaches U1.6 (D32)
- net TOUCH_2: now reaches U1.7 (D33)
- new net: D1.1 (K), R2.1
- new net: J3.2 (Pin_2), R8.2
- new net: D4.1 (K), R5.1
- new net: D2.1 (K), R3.1
- new net: D3.1 (K), R4.1
- new net +3.3V: J2.1 (Pin_1), R1.1, U1.30 (3V3)
Other:
- moved on the sheet: U1

Commit message: working-good music visualization, changing settings of vis to be added
Connections:
- net GND: now also R7.2; no longer R7.1
- net MOTION: now also R7.1, R8.2; no longer R7.2, R8.1
- net at J3.2 (Pin_2): now also R8.1; no longer R8.2
Other:
- note added: "FOR MOTION SENSOR USE ONLY ONE (VOLTAGE)"
- note added: "LDR SENSOR"
- note added: "LED OUTPUT"
- note added: "MCU UNIT"
- note added: "MOTION SENSOR 3.3V"
- note added: "MOTION SENSOR 5V"
- note added: "POWER INPUT"
- note added: "STATUS LEDS"
- note added: "TOUCH_x ROUTED TO PCB PADS"
- moved on the sheet: D1, D2, D3, D4, J1, J2, J3, J4, R1, R2, R3, R4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
